File: pcb/FancyBoard.kicad_pcb (KiCad board)
At the start: 2 copper layers, 336.4 x 114.7 mm, 179 parts, among them J1 Conn_01x02_Socket, SW1 SW_Push_45deg, SW10 SW_Push_45deg, SW11 SW_Push_45deg, SW12 SW_Push_45deg, SW13 SW_Push_45deg, SW14 SW_Push_45deg, SW15 SW_Push_45deg, SW16 SW_Push_45deg, SW17 SW_Push_45deg, SW18 SW_Push_45deg, SW19 SW_Push_45deg, SW2 SW_Push_45deg, SW20 SW_Push_45deg, SW21 SW_Push_45deg, SW22 SW_Push_45deg, SW23 SW_Push_45deg, SW24 SW_Push_45deg, SW25 SW_Push_45deg, SW26 SW_Push_45deg, SW27 SW_Push_45deg, SW28 SW_Push_45deg, SW29 SW_Push_45deg, SW3 SW_Push_45deg, SW30 SW_Push_45deg, SW31 SW_Push_45deg, SW32 SW_Push_45deg, SW33 SW_Push_45deg, SW34 SW_Push_45deg, SW35 SW_Push_45deg, SW36 SW_Push_45deg, SW37 SW_Push_45deg, SW38 SW_Push_45deg, SW39 SW_Push_45deg, SW4 SW_Push_45deg, SW40 SW_Push_45deg, SW41 SW_Push_45deg, SW42 SW_Push_45deg, SW43 SW_Push_45deg, SW44 SW_Push_45deg, SW45 SW_Push_45deg, SW46 SW_Push_45deg, SW47 SW_Push_45deg, SW48 SW_Push_45deg, SW49 SW_Push_45deg, SW5 SW_Push_45deg, SW50 SW_Push_45deg, SW51 SW_Push_45deg, SW52 SW_Push_45deg, SW53 SW_Push_45deg, SW54 SW_Push_45deg, SW55 SW_Push_45deg, SW56 SW_Push_45deg, SW57 SW_Push_45deg, SW58 SW_Push_45deg, SW59 SW_Push_45deg, SW6 SW_Push_45deg, SW60 SW_Push_45deg, SW61 SW_Push_45deg, SW62 SW_Push_45deg, SW63 SW_Push_45deg, SW64 SW_Push_45deg, SW65 SW_Push_45deg, SW66 SW_Push_45deg, SW67 SW_Push_45deg, SW68 SW_Push_45deg, SW69 SW_Push_45deg, SW7 SW_Push_45deg, SW70 SW_Push_45deg, SW71 SW_Push_45deg, SW72 SW_Push_45deg, SW73 SW_Push_45deg, SW74 SW_Push_45deg, SW75 SW_Push_45deg, SW76 SW_Push_45deg, SW77 SW_Push_45deg, SW78 SW_Push_45deg, SW8 SW_Push_45deg, SW9 SW_Push_45deg, SW93 RotaryEncoder_Switch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

Commit message: mostly done routing
Parts:
- moved R1 1.60 mm to (327.7, 136.3)
- moved C6 1.50 mm to (329.2, 136.3)
- moved J1 0.60 mm to (332.6, 108.8)
Connections:
- R10 pad 2: IO18 -> SWITCH_USB
- R11 pad 2: IO9 -> SWITCH_BLE
- SW95 pad 1: IO18 -> SWITCH_USB
- SW95 pad 3: IO9 -> SWITCH_BLE
- U3 pad 9: +3V3 -> GND
- U4 pad 27: unconnected-(U4-GPA6-Pad27) -> SWITCH_USB
- U4 pad 28: unconnected-(U4-GPA7-Pad28) -> SWITCH_BLE
- U4 pad 9: +3V3 -> GND
Routing:
- net COL1: track 106.1 -> 548.3 mm
- net COL2: track 116.0 -> 528.5 mm
- net COL3: track 114.0 -> 499.0 mm
- net COL4: track 139.1 -> 448.7 mm
- net COL5: track 189.6 -> 425.5 mm
- net ROW1: track 281.4 -> 482.5 mm, vias 0 -> 1
- net ROW2: track 281.4 -> 481.6 mm, vias 0 -> 1
- net COL6: track 211.9 -> 403.0 mm
- net COL7: track 194.2 -> 384.5 mm, vias 2 -> 4
- net COL8: track 197.9 -> 372.7 mm, vias 2 -> 4
- net ROW3: track 281.4 -> 443.0 mm, vias 0 -> 1
- net COL9: track 190.5 -> 350.6 mm, vias 4 -> 2
- net COL11: track 91.8 -> 249.1 mm, vias 2 -> 6
- net +3V3: track 0.00 -> 156.7 mm
- net COL14: track 42.0 -> 196.9 mm, vias 0 -> 2
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- added copper zone on B.Cu, net GND
Other:
- board size 336.4 x 114.7 mm -> 338.3 x 116.8 mm

Commit message: pcb done?
Routing:
- net GND: track 0.00 -> 284.6 mm, vias 0 -> 9
- net IO19: track 23.1 -> 26.2 mm, vias 1 -> 2

Commit message: pcb done
Parts:
- SW95: footprint SS-12D00:SS12-D00 -> MSK-12C02:MSK-12C02
- moved D12 1.94 mm to (256.0, 115.2), turned to -90 degrees
- moved D40 1.94 mm to (256.0, 153.2), turned to -90 degrees
- moved D54 1.94 mm to (260.8, 172.3), turned to -90 degrees
- moved D55 1.94 mm to (291.8, 172.3), turned to -90 degrees
- moved D68 1.94 mm to (303.7, 191.3), turned to -90 degrees
- moved D77 1.94 mm to (284.6, 210.4), turned to -90 degrees
- moved D78 1.94 mm to (303.7, 210.4), turned to -90 degrees
- moved D10 1.94 mm to (217.9, 115.2), turned to -90 degrees
- moved D11 1.94 mm to (237.0, 115.2), turned to -90 degrees
- moved D3 1.94 mm to (84.6, 115.2), turned to -90 degrees
- moved D31 1.94 mm to (84.6, 153.2), turned to -90 degrees
- moved D32 1.94 mm to (103.6, 153.2), turned to -90 degrees
- moved D33 1.94 mm to (122.7, 153.2), turned to -90 degrees
- moved D34 1.94 mm to (141.7, 153.2), turned to -90 degrees
- moved D35 1.94 mm to (160.8, 153.2), turned to -90 degrees
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Routing:
- net ROW2: track 481.6 -> 443.1 mm
- net GND: track 284.6 -> 247.3 mm
- net ROW1: track 482.5 -> 456.5 mm
- net ROW3: track 443.0 -> 423.3 mm
- net ROW4: track 411.3 -> 427.2 mm
- net COL8: track 372.7 -> 358.9 mm, vias 4 -> 0
- net IO6: track 75.9 -> 63.3 mm
- net IO7: track 71.7 -> 60.0 mm
- net IO0: track 104.1 -> 114.7 mm
- net IO1: track 112.4 -> 122.8 mm
- net COL14: track 196.9 -> 186.7 mm
- net COL4: track 448.7 -> 439.5 mm, vias 2 -> 0
- net COL3: track 499.0 -> 490.4 mm
- net COL2: track 528.5 -> 520.0 mm
- net SDA: track 109.5 -> 101.2 mm
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Other:
- board text added: "by darsh !!"
